Commit message: trains and stands up

File: segway.urdf (robot description, URDF)
Before this commit: robot segway, 3 links, 2 joints
Links:
- added link battery, mass 0.047; visual cylinder length=0.065 radius=0.009
- added link left_motor_case, mass 0.017; visual box size=0.025 0.015 0.020
- added link right_motor_case, mass 0.017; visual box size=0.025 0.015 0.020
- link chassis: mass 0.026 -> 0.0026
Joints:
- removed joint left_wheel_joint
- removed joint right_wheel_joint
- added joint battery_on_chassis: type fixed, parent chassis, child battery, origin xyz=0 0 -0.032 rpy=0 1.5708 0
- added joint left_drive: type continuous, parent chassis, child left_wheel, origin xyz=-0.048 0.001 -0.021 rpy=0 1.5708 0, axis 0 0 -1
- added joint left_motor_case_joint: type fixed, parent chassis, child left_motor_case, origin xyz=-0.028 0.001 -0.005 rpy=0 0 0
- added joint right_drive: type continuous, parent chassis, child right_wheel, origin xyz=0.048 0.001 -0.021 rpy=0 1.5708 0, axis 0 0 -1
- added joint right_motor_case_joint: type fixed, parent chassis, child right_motor_case, origin xyz=0.028 0.001 -0.005 rpy=0 0 0

Commit message: cleanup env, simplified reward. single script to show model off checkpoints and record a video

File: segway.urdf (robot description, URDF)
Before this commit: robot segway, 6 links, 5 joints
Links:
- added link circuits_link, mass 0.010; visual box size=0.070 0.003 0.015
- added link imu_link, mass 0.002; visual box size=0.015 0.015 0.003
Joints:
- added joint circuits_joint: type fixed, parent chassis, child circuits_link, origin xyz=0 0.005 0.025 rpy=0 0 0
- added joint imu_joint: type fixed, parent chassis, child imu_link, origin xyz=0 0 0.035 rpy=0 0 0

Commit message: Emulate IMU from imu link instead of chassis. Add balance reward besides just upright, minimizing yaw velocity. Add output (pwm, torque) to debug info.

File: segway.urdf (robot description, URDF)
Before this commit: robot segway, 8 links, 7 joints
Links:
- removed link imu_link
- added link imu, mass 0.002; visual box size=0.015 0.015 0.003
Joints:
- joint imu_joint: child imu_link -> imu
